File: Hardware/220vFancontrol/220vFancontrol.sch (KiCad schematic (older format))
At the start: 17 parts, among them Q1 BT136-600, T1 Transformer_1P_1S, U1 MOC3010M, U2 PC817

Commit message: .
Parts:
- added C?: 100nF, symbol Device:C_Small
- added C?: 22pF, symbol Device:C_Small
- C1: value 25v 10uf -> 25v 220uf
- R3: value 10k -> 2.2k
- R4: value 20k -> 5k
Connections:
- net 0-Cross: now also C?.1
- net GND: now also C?.2, C?.2
- net NTC: now also C?.1
Other:
- moved on the sheet: D2, D3, R3, R4, R5, R6, R7, U2
